Commit message: Update models

File: athos_description/robots/pioneer3at_body.xacro (robot description, xacro)
@@ -9,6 +9,6 @@
 	<link name="chassis">
 		<inertial>
-			<mass value="10.0"/>
-			<origin xyz="0 0 0.0"/>
+			<mass value="20.0"/>
+			<origin xyz="0 0 -0.090"/>
 			<inertia ixx="0.3338" ixy="0.0" ixz="0.0"
 				 iyy="0.4783" iyz="0.0"
@@ -18,5 +18,5 @@
 			<origin xyz="0 0 0.0" rpy="0 0 0"/>
 			<geometry name="pioneer_geom">
-				<mesh filename="package://athos_description/meshes/chassis.dae"/>
+				<mesh filename="package://porthos_description/meshes/chassis.dae"/>
 			</geometry>
 			<material name="ChassisRed" />
@@ -25,5 +25,5 @@
 			<origin xyz="0 0 0.0" rpy="0 0 0"/>
 				<geometry>
-					<mesh filename="package://athos_description/meshes/chassis.dae"/>
+					<mesh filename="package://porthos_description/meshes/chassis.dae"/>
 				</geometry>
 		</collision>
@@ -49,5 +49,5 @@
 			<origin xyz="0 0 0" rpy="0 0 0"/>
 			<geometry name="pioneer_geom">
-				<mesh filename="package://athos_description/meshes/top.dae"/>
+				<mesh filename="package://porthos_description/meshes/top.dae"/>
 			</geometry>
 			<material name="TopBlack">
@@ -81,5 +81,5 @@
 			<origin xyz="0 0 0" rpy="0 0 0"/>
 			<geometry name="pioneer_geom">
-				<mesh filename="package://athos_description/meshes/front_sonar.dae"/>
+				<mesh filename="package://porthos_description/meshes/front_sonar.dae"/>
 			</geometry>
 			<material name="SonarYellow">
@@ -112,5 +112,5 @@
 			<origin xyz="0 0 0" rpy="0 0 0"/>
 			<geometry name="pioneer_geom">
-				<mesh filename="package://athos_description/meshes/back_sonar.dae"/>
+				<mesh filename="package://porthos_description/meshes/back_sonar.dae"/>
 			</geometry>
 			<material name="SonarYellow">
@@ -145,5 +145,5 @@
 		<origin xyz="0 0 0" rpy="0 0 0"/>
 		<geometry name="pioneer_geom">
-			<mesh filename="package://athos_description/meshes/axle.dae"/>
+			<mesh filename="package://porthos_description/meshes/axle.dae"/>
 		</geometry>
 		<material name="AxleGrey">
@@ -176,5 +176,5 @@
 		<origin xyz="0 0 0" rpy="0 0 0"/>
 		<geometry name="pioneer_geom">
-			<mesh filename="package://athos_description/meshes/${suffix}_hubcap.dae"/>
+			<mesh filename="package://porthos_description/meshes/${suffix}_hubcap.dae"/>
 		</geometry>
 		<material name="HubcapYellow">
@@ -207,5 +207,5 @@
 		<origin xyz="0 0 0" rpy="0 0 0"/>
 		<geometry name="pioneer_geom">
-			<mesh filename="package://athos_description/meshes/wheel.dae"/>
+			<mesh filename="package://porthos_description/meshes/wheel.dae"/>
 		</geometry>
 		<material name="WheelBlack">
@@ -216,6 +216,6 @@
 		<origin xyz="0 0 0" rpy="${-3.1415927/2} 0 0"/>
 		<geometry>
-	    <!--mesh filename="package://athos_description/meshes/wheel.dae"/-->
-	    <cylinder radius="0.111" length="0.075"/>
+	    <!--mesh filename="package://porthos_description/meshes/wheel.dae"/-->
+	    <cylinder radius="0.110" length="0.035"/>
 		</geometry>
 	</collision>
@@ -246,5 +246,5 @@
 		<origin xyz="0 0 0" rpy="0 0 0"/>
 		<geometry name="pioneer_geom">
-			<mesh filename="package://athos_description/meshes/axle.dae"/>
+			<mesh filename="package://porthos_description/meshes/axle.dae"/>
 		</geometry>
 		<material name="AxleGrey">
@@ -255,5 +255,5 @@
 		<origin xyz="0 0 0" rpy="0 0 0"/>
 		<geometry>
-			<mesh filename="package://athos_description/meshes/axle.dae"/>
+			<mesh filename="package://porthos_description/meshes/axle.dae"/>
 		</geometry>
 	</collision>
@@ -277,5 +277,5 @@
 		<origin xyz="0 0 0" rpy="0 0 0"/>
 		<geometry name="pioneer_geom">
-			<mesh filename="package://athos_description/meshes/${suffix}_hubcap.dae"/>
+			<mesh filename="package://porthos_description/meshes/${suffix}_hubcap.dae"/>
 		</geometry>
 		<material name="HubcapYellow"/>
@@ -284,5 +284,5 @@
 		<origin xyz="0 0 0" rpy="0 0 0"/>
 		<geometry>
-			<mesh filename="package://athos_description/meshes/${suffix}_hubcap.dae"/>
+			<mesh filename="package://porthos_description/meshes/${suffix}_hubcap.dae"/>
 		</geometry>
 	</collision>
@@ -306,5 +306,5 @@
 		<origin xyz="0 0 0" rpy="0 0 0"/>
 		<geometry name="pioneer_geom">
-			<mesh filename="package://athos_description/meshes/wheel.dae"/>
+			<mesh filename="package://porthos_description/meshes/wheel.dae"/>
 		</geometry>
 		<material name="WheelBlack"/>
@@ -313,6 +313,6 @@
 		<origin xyz="0 0 0" rpy="${-3.1415927/2} 0 0"/>
 		<geometry>
-	    <!--mesh filename="package://athos_description/meshes/wheel.dae"/-->
-	    <cylinder radius="0.111" length="0.075"/>
+	    <!--mesh filename="package://porthos_description/meshes/wheel.dae"/-->
+	    <cylinder radius="0.110" length="0.035"/>
 		</geometry>
 	</collision>
@@ -334,6 +334,6 @@
     <kd>100.0</kd>
     <mu1>10.0</mu1>
-    <mu2>1.0</mu2>
-    <fdir1>0 1 0</fdir1> <!-- is this correct? -->
+    <mu2>0.1</mu2>
+    <fdir1>1 0 0</fdir1> <!-- is this correct? -->
     <maxVel>1.0</maxVel>
     <minDepth>0.00</minDepth>
@@ -343,6 +343,6 @@
     <kd>100.0</kd>
     <mu1>10.0</mu1>
-    <mu2>1.0</mu2>
-    <fdir1>0 1 0</fdir1> <!-- is this correct? -->
+    <mu2>0.1</mu2>
+    <fdir1>1 0 0</fdir1> <!-- is this correct? -->
     <maxVel>1.0</maxVel>
     <minDepth>0.00</minDepth>
@@ -354,5 +354,5 @@
       <robotNamespace></robotNamespace>
       <jointName>p3at_front_left_wheel_joint, p3at_front_right_wheel_joint, p3at_back_left_wheel_joint, p3at_back_right_wheel_joint</jointName>
-      <updateRate>50.0</updateRate>
+      <updateRate>10.0</updateRate>
       <alwaysOn>true</alwaysOn>
     </plugin>
@@ -361,5 +361,4 @@
   <plugin name="skid_steer_drive_controller" filename="libgazebo_ros_skid_steer_drive.so">
     <updateRate>50.0</updateRate>
-    <!-- <robotNamespace>/</robotNamespace> -->
     <leftFrontJoint>p3at_front_left_wheel_joint</leftFrontJoint>
     <rightFrontJoint>p3at_front_right_wheel_joint</rightFrontJoint>
@@ -368,11 +367,19 @@
     <odometryTopic>pose</odometryTopic>
     <wheelSeparation>0.4</wheelSeparation>
-    <wheelDiameter>0.215</wheelDiameter>
+    <wheelDiameter>0.220</wheelDiameter>
+    <covariance_x>1</covariance_x>
+    <covariance_y>1</covariance_y>
+    <covariance_yaw>1</covariance_yaw>
     <robotBaseFrame>base_link</robotBaseFrame>
     <commandTopic>cmd_vel</commandTopic>
     <odometryFrame>odom</odometryFrame>
     <broadcastTF>1</broadcastTF>
-    <torque>200</torque>
+    <wheel_accel>1.8</wheel_accel>
+    <torque>5</torque>
     <topicName>cmd_vel</topicName>
+    <alpha1>0.001</alpha1>
+    <alpha2>0.001</alpha2>
+    <alpha3>0.001</alpha3>
+    <alpha4>0.001</alpha4>
   </plugin>
 </gazebo>

File: athos_description/robots/suporte_athos_description.urdf (robot description, URDF)
Before this commit: robot suporte_athos_description, 10 links, 9 joints
Links:
- removed link tv
- link arm_control_box: mass 1.88580869219064 -> 0.45
- link suporte_base: mass 1 -> 0.5
Joints:
- removed joint suporte2tv
